File: board/SleekAVC64.kicad_pcb (KiCad board)
At the start: 2 copper layers, 36.8 x 25.4 mm, 10 parts, among them J1 Mini-DIN-4, J2 SV80, J3 LEFT, J4 RIGHT, J5 CVBS, SW1 SW_SPDT

Commit message: Adding case and media
Signed-off-by: Martin Matyas <martin.matyas@gmail.com>
Other:
- board text added: "1.0.0"
- board text removed: "1.0"
Changed lines of the file:
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@@
 			(drillshape 0)
 			(scaleselection 1)
-			(outputdirectory "")
+			(outputdirectory ".")
 		)
 	)
@@
 		)
 	)
-	(gr_text "1.0"
-		(at 149.86 110.49 0)
+	(gr_text "1.0.0"
+		(at 153.67 110.49 0)
 		(layer "B.SilkS")
 		(effects
@@
 			(justify left bottom mirror)
 		)
-		(render_cache "1.0" 0
+		(render_cache "1.0.0" 0
 			(polygon
 				(pts
-					(xy 149.86 110.15) (xy 149.86 109.799755) (xy 149.32987 109.799755) (xy 149.32987 108.749511) (xy 149.594752 108.749511)
-					(xy 149.594752 108.399267) (xy 149.32987 108.399267) (xy 149.32987 107.711479) (xy 148.80487 107.711479)
-					(xy 148.80487 109.799755) (xy 148.28903 109.799755) (xy 148.28903 110.15)
+					(xy 153.67 110.15) (xy 153.67 109.799755) (xy 153.13987 109.799755) (xy 153.13987 108.749511) (xy 153.404752 108.749511)
+					(xy 153.404752 108.399267) (xy 153.13987 108.399267) (xy 153.13987 107.711479) (xy 152.61487 107.711479)
+					(xy 152.61487 109.799755) (xy 152.09903 109.799755) (xy 152.09903 110.15)
 				)
 			)
 			(polygon
 				(pts
-					(xy 148.022316 110.15) (xy 148.022316 109.462212) (xy 147.497316 109.462212) (xy 147.497316 110.15)
+					(xy 151.832316 110.15) (xy 151.832316 109.462212) (xy 151.307316 109.462212) (xy 151.307316 110.15)
 				)
 			)
 			(polygon
 				(pts
-					(xy 146.977445 108.055373) (xy 147.235366 108.055373) (xy 147.235366 109.806106) (xy 146.977445 109.806106)
-					(xy 146.977445 110.15) (xy 145.922316 110.15) (xy 145.922316 109.806106) (xy 145.664396 109.806106)
-					(xy 145.664396 109.799755) (xy 146.189396 109.799755) (xy 146.710366 109.799755) (xy 146.710366 109.093405)
-					(xy 146.449881 109.093405) (xy 146.449881 108.749511) (xy 146.189396 108.749511) (xy 146.189396 109.799755)
-					(xy 145.664396 109.799755) (xy 145.664396 108.399267) (xy 146.189396 108.399267) (xy 146.449881 108.399267)
-					(xy 146.449881 108.743161) (xy 146.710366 108.743161) (xy 146.710366 108.061723) (xy 146.189396 108.061723)
-					(xy 146.189396 108.399267) (xy 145.664396 108.399267) (xy 145.664396 108.055373) (xy 145.922316 108.055373)
-					(xy 145.922316 107.711479) (xy 146.977445 107.711479)
+					(xy 150.787445 108.055373) (xy 151.045366 108.055373) (xy 151.045366 109.806106) (xy 150.787445 109.806106)
+					(xy 150.787445 110.15) (xy 149.732316 110.15) (xy 149.732316 109.806106) (xy 149.474396 109.806106)
+					(xy 149.474396 109.799755) (xy 149.999396 109.799755) (xy 150.520366 109.799755) (xy 150.520366 109.093405)
+					(xy 150.259881 109.093405) (xy 150.259881 108.749511) (xy 149.999396 108.749511) (xy 149.999396 109.799755)
+					(xy 149.474396 109.799755) (xy 149.474396 108.399267) (xy 149.999396 108.399267) (xy 150.259881 108.399267)
+					(xy 150.259881 108.743161) (xy 150.520366 108.743161) (xy 150.520366 108.061723) (xy 149.999396 108.061723)
+					(xy 149.999396 108.399267) (xy 149.474396 108.399267) (xy 149.474396 108.055373) (xy 149.732316 108.055373)
+					(xy 149.732316 107.711479) (xy 150.787445 107.711479)
+				)
+			)
+			(polygon
+				(pts
+					(xy 149.207683 110.15) (xy 149.207683 109.462212) (xy 148.682683 109.462212) (xy 148.682683 110.15)
+				)
+			)
+			(polygon
+				(pts
+					(xy 148.162812 108.055373) (xy 148.420732 108.055373) (xy 148.420732 109.806106) (xy 148.162812 109.806106)
+					(xy 148.162812 110.15) (xy 147.107683 110.15) (xy 147.107683 109.806106) (xy 146.849762 109.806106)
+					(xy 146.849762 109.799755) (xy 147.374762 109.799755) (xy 147.895732 109.799755) (xy 147.895732 109.093405)
+					(xy 147.635247 109.093405) (xy 147.635247 108.749511) (xy 147.374762 108.749511) (xy 147.374762 109.799755)
+					(xy 146.849762 109.799755) (xy 146.849762 108.399267) (xy 147.374762 108.399267) (xy 147.635247 108.399267)
+					(xy 147.635247 108.743161) (xy 147.895732 108.743161) (xy 147.895732 108.061723) (xy 147.374762 108.061723)
+					(xy 147.374762 108.399267) (xy 146.849762 108.399267) (xy 146.849762 108.055373) (xy 147.107683 108.055373)
+					(xy 147.107683 107.711479) (xy 148.162812 107.711479)
 				)
 			)
